File: Carrier-Board.kicad_pcb (KiCad board)
At the start: 4 copper layers, 92 x 96 mm, 11 parts, among them J1 CONN_3-6318491-6, U9 MSATA-Socket

Commit message: SF
Parts:
- added J2: 0532610671, MOLEX_0532610671, F.Cu at (48.5, 57.9)
Connections:
- J1 pad 116: (no net) -> Net-(J1-Pad116)
- J1 pad 117: (no net) -> Net-(J1-Pad117)
- J1 pad 118: (no net) -> Net-(J1-Pad118)
- J1 pad 119: (no net) -> Net-(J1-Pad119)
- J1 pad 120: (no net) -> Net-(J1-Pad120)
Changed lines of the file:
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@@
 (kicad_pcb (version 4) (host pcbnew 4.0.7)
   (general
-    (links 68)
-    (no_connects 68)
-    (area 71.837143 -42.371452 174.170001 124.545)
+    (links 173)
+    (no_connects 173)
+    (area 0 0 0 0)
     (thickness 1.6)
     (drawings 2)
     (tracks 1)
     (zones 0)
-    (modules 11)
-    (nets 312)
+    (modules 12)
+    (nets 324)
   )
   (page A4)
@@
   (net 310 GNDREF)
   (net 311 mCOM_GND)
+  (net 312 "Net-(J1-Pad120)")
+  (net 313 "Net-(J1-Pad119)")
+  (net 314 "Net-(J1-Pad118)")
+  (net 315 "Net-(J1-Pad117)")
+  (net 316 "Net-(J1-Pad116)")
+  (net 317 "Net-(J2-Pad1)")
+  (net 318 "Net-(J2-Pad2)")
+  (net 319 "Net-(J2-Pad3)")
+  (net 320 "Net-(J2-Pad4)")
+  (net 321 "Net-(J2-Pad5)")
+  (net 322 "Net-(J2-Pad6)")
+  (net 323 "Net-(J2-PadS1)")
   (net_class Default "This is the default net class."
     (clearance 0.2)
@@
     (add_net "Net-(J1-Pad114)")
     (add_net "Net-(J1-Pad115)")
+    (add_net "Net-(J1-Pad116)")
+    (add_net "Net-(J1-Pad117)")
+    (add_net "Net-(J1-Pad118)")
+    (add_net "Net-(J1-Pad119)")
+    (add_net "Net-(J1-Pad120)")
     (add_net "Net-(J1-Pad123)")
     (add_net "Net-(J1-Pad124)")
@@
     (add_net "Net-(J1-Pad91)")
     (add_net "Net-(J1-Pad96)")
+    (add_net "Net-(J2-Pad1)")
+    (add_net "Net-(J2-Pad2)")
+    (add_net "Net-(J2-Pad3)")
+    (add_net "Net-(J2-Pad4)")
+    (add_net "Net-(J2-Pad5)")
+    (add_net "Net-(J2-Pad6)")
+    (add_net "Net-(J2-PadS1)")
     (add_net "Net-(J3-Pad1)")
     (add_net "Net-(J3-Pad10)")
@@
     (pad 121 smd rect (at 56.732997 2.8338) (size 0.3302 1.1938) (layers F.Cu F.Paste F.Mask)
       (net 311 mCOM_GND))
-    (pad 120 smd rect (at 57.232996 2.8338) (size 0.3302 1.1938) (layers F.Cu F.Paste F.Mask))
-    (pad 119 smd rect (at 57.732997 2.8338) (size 0.3302 1.1938) (layers F.Cu F.Paste F.Mask))
-    (pad 118 smd rect (at 58.232996 2.8338) (size 0.3302 1.1938) (layers F.Cu F.Paste F.Mask))
-    (pad 117 smd rect (at 58.732998 2.8338) (size 0.3302 1.1938) (layers F.Cu F.Paste F.Mask))
-    (pad 116 smd rect (at 59.232997 2.8338) (size 0.3302 1.1938) (layers F.Cu F.Paste F.Mask))
+    (pad 120 smd rect (at 57.232996 2.8338) (size 0.3302 1.1938) (layers F.Cu F.Paste F.Mask)
+      (net 312 "Net-(J1-Pad120)"))
+    (pad 119 smd rect (at 57.732997 2.8338) (size 0.3302 1.1938) (layers F.Cu F.Paste F.Mask)
+      (net 313 "Net-(J1-Pad119)"))
+    (pad 118 smd rect (at 58.232996 2.8338) (size 0.3302 1.1938) (layers F.Cu F.Paste F.Mask)
+      (net 314 "Net-(J1-Pad118)"))
+    (pad 117 smd rect (at 58.732998 2.8338) (size 0.3302 1.1938) (layers F.Cu F.Paste F.Mask)
+      (net 315 "Net-(J1-Pad117)"))
+    (pad 116 smd rect (at 59.232997 2.8338) (size 0.3302 1.1938) (layers F.Cu F.Paste F.Mask)
+      (net 316 "Net-(J1-Pad116)"))
     (pad 115 smd rect (at 59.732996 2.8338) (size 0.3302 1.1938) (layers F.Cu F.Paste F.Mask)
       (net 108 "Net-(J1-Pad115)"))
@@
       (net 281 "Net-(J5-Pad52)"))
   )
+  (module MOLEX_0532610671 (layer F.Cu)
+    (at 48.55 57.9)
+    (attr smd)
+    (fp_text reference J2 (at -2.94812 -1.70953) (layer F.SilkS)
+      (effects (font (size 0.32119 0.32119) (thickness 0.05)))
+    )
+    (fp_text value 0532610671 (at -2.73998 5.77139) (layer F.SilkS)
+      (effects (font (size 0.320699 0.320699) (thickness 0.05)))
+    )
+    (fp_line (start -6.125 0.8) (end -6.125 5) (layer Dwgs.User) (width 0.127))
+    (fp_line (start -6.125 5) (end 6.125 5) (layer Dwgs.User) (width 0.127))
+    (fp_line (start 6.125 5) (end 6.125 0.8) (layer Dwgs.User) (width 0.127))
+    (fp_line (start 6.125 0.8) (end -6.125 0.8) (layer Dwgs.User) (width 0.127))
+    (fp_line (start -6.125 0.8) (end -3.75 0.8) (layer F.SilkS) (width 0.127))
+    (fp_line (start -6.125 0.8) (end -6.125 1.25) (layer F.SilkS) (width 0.127))
+    (fp_line (start -6.125 5) (end 6.125 5) (layer F.SilkS) (width 0.127))
+    (fp_line (start 3.75 0.8) (end 6.125 0.8) (layer F.SilkS) (width 0.127))
+    (fp_line (start 6.125 0.8) (end 6.125 1.25) (layer F.SilkS) (width 0.127))
+    (fp_line (start -3.775 0.55) (end -3.775 -1.05) (layer Dwgs.User) (width 0.05))
+    (fp_line (start -3.775 -1.05) (end 3.775 -1.05) (layer Dwgs.User) (width 0.05))
+    (fp_line (start 3.775 -1.05) (end 3.775 0.55) (layer Dwgs.User) (width 0.05))
+    (fp_line (start 3.775 0.55) (end 6.375 0.55) (layer Dwgs.User) (width 0.05))
+    (fp_line (start 6.375 0.55) (end 6.375 1.15) (layer Dwgs.User) (width 0.05))
+    (fp_line (start 6.375 1.15) (end 6.975 1.15) (layer Dwgs.User) (width 0.05))
+    (fp_line (start 6.975 1.15) (end 6.975 5.25) (layer Dwgs.User) (width 0.05))
+    (fp_line (start 6.975 5.25) (end -6.975 5.25) (layer Dwgs.User) (width 0.05))
+    (fp_line (start -6.975 5.25) (end -6.975 1.15) (layer Dwgs.User) (width 0.05))
+    (fp_line (start -6.975 1.15) (end -6.375 1.15) (layer Dwgs.User) (width 0.05))
+    (fp_line (start -6.375 1.15) (end -6.375 0.55) (layer Dwgs.User) (width 0.05))
+    (fp_line (start -6.375 0.55) (end -3.775 0.55) (layer Dwgs.User) (width 0.05))
+    (fp_circle (center -3.125 -1.3) (end -3.025 -1.3) (layer F.SilkS) (width 0.2))
+    (pad 1 smd rect (at -3.125 0 90) (size 1.6 0.8) (layers F.Cu F.Paste F.Mask)
+      (net 317 "Net-(J2-Pad1)"))
+    (pad 2 smd rect (at -1.875 0 90) (size 1.6 0.8) (layers F.Cu F.Paste F.Mask)
+      (net 318 "Net-(J2-Pad2)"))
+    (pad 3 smd rect (at -0.625 0 90) (size 1.6 0.8) (layers F.Cu F.Paste F.Mask)
+      (net 319 "Net-(J2-Pad3)"))
+    (pad 4 smd rect (at 0.625 0 90) (size 1.6 0.8) (layers F.Cu F.Paste F.Mask)
+      (net 320 "Net-(J2-Pad4)"))
+    (pad 5 smd rect (at 1.875 0 90) (size 1.6 0.8) (layers F.Cu F.Paste F.Mask)
+      (net 321 "Net-(J2-Pad5)"))
+    (pad 6 smd rect (at 3.125 0 90) (size 1.6 0.8) (layers F.Cu F.Paste F.Mask)
+      (net 322 "Net-(J2-Pad6)"))
+    (pad S1 smd rect (at -5.675 2.9 90) (size 3 2.1) (layers F.Cu F.Paste F.Mask)
+      (net 323 "Net-(J2-PadS1)"))
+    (pad S2 smd rect (at 5.675 2.9 90) (size 3 2.1) (layers F.Cu F.Paste F.Mask)
+      (net 323 "Net-(J2-PadS1)"))
+  )
   (gr_text "S/N: 00000000" (at 113.25 107) (layer B.SilkS)

Commit message: added connecttos in lib
Routing:
- added copper zone on B.Cu, net (none)
Changed lines of the file:
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@@
 (kicad_pcb (version 4) (host pcbnew 4.0.7)
   (general
-    (links 173)
-    (no_connects 173)
-    (area 0 0 0 0)
+    (links 69)
+    (no_connects 69)
+    (area 41.349999 -42.371452 174.170001 124.545)
     (thickness 1.6)
     (drawings 2)
@@
   )
   (segment (start 162.08 63.13) (end 162.08 63.71) (width 0.2) (layer F.Cu) (net 310))
+  (zone (net 0) (net_name "") (layer B.Cu) (hatch edge 0.508)
+    (connect_pads (clearance 0.8))
+    (min_thickness 0.254)
+    (fill yes (arc_segments 16) (thermal_gap 0.508) (thermal_bridge_width 0.508))
+    (polygon
+      (pts
+        (xy 110.395 55.25) (xy 116.175 55.26) (xy 116.185 61.03) (xy 110.395 61.04) (xy 110.415 55.25)
+      )
+    )
+  )
+  (zone (net 0) (net_name "") (layer B.Cu) (hatch edge 0.508)
+    (connect_pads (clearance 0.8))
+    (min_thickness 0.254)
+    (fill yes (arc_segments 16) (thermal_gap 0.508) (thermal_bridge_width 0.508))
+    (polygon
+      (pts
+        (xy 110.40343 79.472545) (xy 116.18343 79.482545) (xy 116.19343 85.252545) (xy 110.40343 85.262545) (xy 110.42343 79.472545)
+      )
+    )
+  )
 )

Commit message: ADSFM
Parts:
- added J3: 53261-0771, 53261-0771, F.Cu at (214.1, 8.32)
- added J4: 53261-1071, 532611071, F.Cu at (217.0, 2.48)
- added P1: 0532610471, MOLEX_0532610471, F.Cu at (228.6, 9.57)
- added P10: 0532610471, MOLEX_0532610471, F.Cu at (254.2, 11.4)
- added P11: 0532610471, MOLEX_0532610471, F.Cu at (239.1, 31.9)
- added P12: 0532610471, MOLEX_0532610471, F.Cu at (274.5, 1.16)
- added P13: 0532610471, MOLEX_0532610471, F.Cu at (252.0, 21.6)
- added P14: 0532610471, MOLEX_0532610471, F.Cu at (267.1, 11.4)
- added P2: 0532610471, MOLEX_0532610471, F.Cu at (213.5, 25.9)
- added P3: 0532610471, MOLEX_0532610471, F.Cu at (248.8, 1.16)
- added P4: 0532610471, MOLEX_0532610471, F.Cu at (226.3, 19.8)
- added P5: 0532610471, MOLEX_0532610471, F.Cu at (241.4, 11.4)
- added P6: 0532610471, MOLEX_0532610471, F.Cu at (226.3, 30.0)
- added P7: 0532610471, MOLEX_0532610471, F.Cu at (213.5, 15.7)
- added P8: 0532610471, MOLEX_0532610471, F.Cu at (261.6, 1.16)
- added P9: 0532610471, MOLEX_0532610471, F.Cu at (239.1, 21.6)
- H1: value Conn_02x26_Odd_Even -> H1
- H2: value Conn_02x26_Odd_Even -> H2
- moved J2 194.8 mm to (234.7, 0.48)
Connections:
- net Net-(J3-Pad10) renamed SW2_12v
- net Net-(J3-Pad11) renamed SW3_BatV
- net Net-(J3-Pad12) renamed SW4_BatV
- net Net-(J3-Pad13) renamed SW5_5v
- net Net-(J3-Pad15) renamed SW6_5v
- net Net-(J3-Pad16) renamed SW7_5v
- net Net-(J3-Pad18) renamed SW8_3V3
- net Net-(J3-Pad19) renamed SW9_3V3
- net Net-(J3-Pad20) renamed SW10_3V3
- net Net-(J3-Pad31) renamed AGND
- net Net-(J3-Pad8) renamed SW1_12v
- net Net-(J5-Pad1) renamed CAN_L
- net Net-(J5-Pad10) renamed * GPIO PH11
- net Net-(J5-Pad13) renamed * ADC1_IN4 (PC4)
- net Net-(J5-Pad14) renamed * ADC1_IN8 (PC5)
- net Net-(J5-Pad15) renamed * ADC1_IN5 (PB1)
- net Net-(J5-Pad16) renamed * ADC1_IN9 (PB0)
- net Net-(J5-Pad17) renamed * UHF radio UART2_RX / ** UART2_TX
- net Net-(J5-Pad18) renamed * UHF radio UART2_TX / ** UART2_RX
- net Net-(J5-Pad2) renamed GPS_PPS signal output
- net Net-(J5-Pad3) renamed CAN_H
- net Net-(J5-Pad32) renamed 5VUSB_CHG
- net Net-(J5-Pad41) renamed * I2C3_SDA
- net Net-(J5-Pad43) renamed * I2C3_SCL
- net Net-(J5-Pad47) renamed 5 V Reaction wheels power supply (default option)
- net Net-(J5-Pad48) renamed 3.3 V 3C2 board power supply (default option)
- net Net-(J5-Pad5) renamed *GPIO_PA10
- net Net-(J5-Pad7) renamed * GPIO_PH6
- net Net-(J5-Pad8) renamed * GPIO_PH9
- net Net-(J5-Pad9) renamed * GPIO PH10
- H2 pad 14: Net-(J3-Pad14) -> GND
- H2 pad 17: Net-(J3-Pad17) -> GND
- H2 pad 21: Net-(J3-Pad21) -> GND
- H2 pad 22: Net-(J3-Pad22) -> GND
- H2 pad 23: Net-(J3-Pad23) -> 12V
- H2 pad 24: Net-(J3-Pad24) -> 12V
- H2 pad 25: Net-(J3-Pad25) -> 5V
- H2 pad 26: Net-(J3-Pad26) -> 5V
- H2 pad 27: Net-(J3-Pad27) -> 3V3
- H2 pad 28: Net-(J3-Pad28) -> 3V3
- H2 pad 29: Net-(J3-Pad29) -> GND
- H2 pad 30: Net-(J3-Pad30) -> GND
- H2 pad 32: Net-(J3-Pad32) -> GND
- H2 pad 33: Net-(J3-Pad33) -> DNU
- H2 pad 34: Net-(J3-Pad34) -> DNU
- H2 pad 35: Net-(J3-Pad35) -> PCM_IN
- H2 pad 36: Net-(J3-Pad36) -> PCM_IN
- H2 pad 37: Net-(J3-Pad37) -> DNU
- H2 pad 38: Net-(J3-Pad38) -> DNU
- H2 pad 39: Net-(J3-Pad39) -> DNU
- H2 pad 40: Net-(J3-Pad40) -> DNU
- H2 pad 41: Net-(J3-Pad41) -> BCR_OUT
- H2 pad 42: Net-(J3-Pad42) -> BCR_OUT
- H2 pad 43: Net-(J3-Pad43) -> BCR_OUT
- H2 pad 44: Net-(J3-Pad44) -> BCR_OUT
- H2 pad 45: Net-(J3-Pad45) -> BatV
- H2 pad 46: Net-(J3-Pad46) -> BatV
- H2 pad 47: Net-(J3-Pad47) -> GND
- H2 pad 48: Net-(J3-Pad48) -> GND
- H2 pad 9: Net-(J3-Pad9) -> GND
Routing:
- removed copper zone on B.Cu, net (none)
